Commit message: aha

File: install/linorobot2_description/share/linorobot2_description/urdf/4wd_properties.urdf.xacro (robot description, xacro)
@@ -1,8 +1,8 @@
 <?xml version="1.0"?>
 <robot xmlns:xacro="http://ros.org/wiki/xacro">
-  <xacro:property name="base_length" value="0.445" />
-  <xacro:property name="base_width" value="0.200" />
-  <xacro:property name="base_height" value="0.129" />
-  <xacro:property name="base_mass" value="10" />
+  <xacro:property name="base_length" value="0.290" />
+  <xacro:property name="base_width" value="0.230" />
+  <xacro:property name="base_height" value="0.330" />
+  <xacro:property name="base_mass" value="58" />
   <xacro:property name="wheel_radius" value="0.07162" />
   <xacro:property name="wheel_width" value="0.05" />
